Commit message: Enable gazebo simulation

File: src/jetrover_description/urdf/car_acker.urdf.xacro (robot description, xacro)
@@ -194,5 +194,5 @@
   <joint
     name="wheel_left_back_joint"
-    type="fixed">
+    type="continuous">
     <origin
       xyz="0.106753653016542 -0.0920004072996187 -0.0658214520621466"
@@ -203,5 +203,5 @@
       link="wheel_left_back_link" />
     <axis
-      xyz="0 0 0" />
+      xyz="0 1 0" />
   </joint>
   <!-- 右前轮 -->
@@ -296,5 +296,5 @@
   <joint
     name="wheel_right_back_joint"
-    type="fixed">
+    type="continuous">
     <origin
       xyz="0.10675 0.091848 -0.065821"
@@ -305,5 +305,6 @@
       link="wheel_right_back_link" />
     <axis
-      xyz="0 0 0" />
-  </joint>
+      xyz="0 1 0" />
+  </joint>
+  <!-- <xacro:include filename="$(find jetrover_description)/gazebo/car_acker_gazebo.xacro" /> -->
 </robot>
