Commit message: Fully understand the URDF modeling files

File: src/jetrover_description/urdf/arm.urdf.xacro (robot description, xacro)
@@ -2,4 +2,5 @@
 <robot name="arm" xmlns:xacro="http://ros.org/wiki/xacro">
   <xacro:property name="M_PI"   value="3.1415926535897931"/>
+  <!-- 第一节机械臂本体 -->
   <link
     name="link1">
@@ -38,4 +39,5 @@
     </collision>
   </link>
+  <!-- 伺服电机1 -->
   <link
     name="servo_link1">
@@ -74,4 +76,5 @@
     </collision>
   </link>
+  <!-- 第一节机械臂和伺服电机1 联结 -->
   <joint
     name="servo_joint1"
@@ -87,4 +90,5 @@
       xyz="0 0 0" />
   </joint>
+  <!-- 第二节机械臂本体 -->
   <link
     name="link2">
@@ -123,4 +127,5 @@
     </collision>
   </link>
+  <!-- 第二节机械臂和伺服电机1 联结 -->
   <joint
     name="joint2"
@@ -141,4 +146,5 @@
       velocity="10" />
   </joint>
+  <!-- 第三节机械臂本体 -->
   <link
     name="link3">
@@ -177,4 +183,5 @@
     </collision>
   </link>
+  <!-- 第三节机械臂本体和第二节机械臂本体 联结 -->
   <joint
     name="joint3"
@@ -195,4 +202,5 @@
       velocity="10" />
   </joint>
+  <!-- 第四节机械臂本体 -->
   <link
     name="link4">
@@ -231,4 +239,5 @@
     </collision>
   </link>
+  <!-- 第三节机械臂和第四节机械臂 联结 -->
   <joint
     name="joint4"
@@ -249,4 +258,5 @@
       velocity="10" />
   </joint>
+  <!-- 伺服电机2 -->
   <link
     name="servo_link2">
@@ -285,4 +295,5 @@
     </collision>
   </link>
+  <!-- 第四节机械臂和伺服电机2 联结 -->
   <joint
     name="servo_joint2"
@@ -298,4 +309,5 @@
       xyz="0 0 0" />
   </joint>
+  <!-- 夹爪旋转垫片 -->
   <link
     name="link5">
@@ -334,4 +346,5 @@
     </collision>
   </link>
+  <!-- 夹爪旋转垫片和伺服电机2 联结 -->
   <joint
     name="joint5"
@@ -352,4 +365,5 @@
       velocity="10" />
   </joint>
+  <!-- 夹爪底座 -->
   <link
     name="gripper_link">
@@ -388,4 +402,5 @@
     </collision>
   </link>
+  <!-- 夹爪底座和夹爪旋转垫片 联结 -->
   <joint
     name="gripper_joint"
@@ -401,6 +416,7 @@
       xyz="0 0 0" />
   </joint>
-  <!-- end effector link -->
+  <!-- 末端执行器（坐标系） -->
   <link name="end_effector_link" />
+  <!-- 末端执行器（坐标系）和夹爪旋转垫片 联结 -->
   <joint name="end_effector_joint" type="fixed">
     <origin xyz="0 0 0.08" rpy="0 0 0"/>

File: src/jetrover_description/urdf/car_acker.urdf.xacro (robot description, xacro)
@@ -1,16 +1,17 @@
 <?xml version="1.0" encoding="utf-8"?>
-<robot name="jetrover" xmlns:xacro="http://ros.org/wiki/xacro" >
-  <xacro:property name="M_PI"               value="3.1415926535897931"/>
-  <link name="base_footprint"/>
-  <xacro:property name="base_link_mass"     value="1.6" />
-  <xacro:property name="base_link_w"        value="0.30"/>
-  <xacro:property name="base_link_h"        value="0.15"/>
-  <xacro:property name="base_link_d"        value="0.10"/>
+<robot name="jetrover" xmlns:xacro="http://ros.org/wiki/xacro">
+  <xacro:property name="M_PI" value="3.1415926535897931" />
+  <link name="base_footprint" />
+  <xacro:property name="base_link_mass" value="1.6" />
+  <xacro:property name="base_link_w" value="0.30" />
+  <xacro:property name="base_link_h" value="0.15" />
+  <xacro:property name="base_link_d" value="0.10" />
+  <!-- 车底钢板和垂直投影 联结 -->
   <joint name="base_joint" type="fixed">
-    <parent link="base_footprint"/>
-    <child link="base_link"/>
-    <origin xyz="0.0 0.0 ${0.05 + 0.0654867643253843}" rpy="0 0 0"/>
-  </joint>
-  <link name="w_link"/>
+    <parent link="base_footprint" />   <!-- 机器人垂直投影到地面的坐标系 -->
+    <child link="base_link" />
+    <origin xyz="0.0 0.0 ${0.05 + 0.0654867643253843}" rpy="0 0 0" />
+  </joint>
+  <link name="w_link" />
   <joint
     name="w_joint"
@@ -26,7 +27,9 @@
       xyz="0 0 0" />
   </joint>
+  <!-- 车底钢板 -->
   <link
     name="base_link">
-    <xacro:box_inertial m="${base_link_mass}" w="${base_link_w}" h="${base_link_h}" d="${base_link_d}" x="0" y="0" z="-0.15" />
+    <xacro:box_inertial m="${base_link_mass}" w="${base_link_w}" h="${base_link_h}"
+      d="${base_link_d}" x="0" y="0" z="-0.15" />
     <visual>
       <origin
@@ -37,5 +40,5 @@
           filename="package://jetrover_description/meshes/acker/base_link.stl" />
       </geometry>
-      <material name="black"/>
+      <material name="black" />
     </visual>
     <collision>
@@ -49,4 +52,5 @@
     </collision>
   </link>
+  <!-- 车底中间层钢板 -->
   <link
     name="base_green_link">
@@ -73,5 +77,5 @@
           filename="package://jetrover_description/meshes/acker/base_green_link.stl" />
       </geometry>
-      <material name="green"/>
+      <material name="green" />
     </visual>
     <collision>
@@ -85,4 +89,5 @@
     </collision>
   </link>
+  <!-- 车底钢板 中间夹层钢板 联结 -->
   <joint
     name="base_green_joint"
@@ -98,4 +103,5 @@
       xyz="0 0 0" />
   </joint>
+  <!-- 左前轮 -->
   <link
     name="wheel_left_front_link">
@@ -122,5 +128,5 @@
           filename="package://jetrover_description/meshes/acker/wheel_left_front_link.stl" />
       </geometry>
-      <material name="black"/>
+      <material name="black" />
     </visual>
     <collision>
@@ -134,4 +140,5 @@
     </collision>
   </link>
+  <!-- 左前轮和底部钢板 联结 -->
   <joint
     name="wheel_left_front_joint"
@@ -147,4 +154,5 @@
       xyz="0 0 0" />
   </joint>
+  <!-- 左后轮 -->
   <link
     name="wheel_left_back_link">
@@ -171,5 +179,5 @@
           filename="package://jetrover_description/meshes/acker/wheel_left_back_link.stl" />
       </geometry>
-      <material name="black"/>
+      <material name="black" />
     </visual>
     <collision>
@@ -183,4 +191,5 @@
     </collision>
   </link>
+  <!-- 左后轮和底部钢板 联结 -->
   <joint
     name="wheel_left_back_joint"
@@ -196,4 +205,5 @@
       xyz="0 0 0" />
   </joint>
+  <!-- 右前轮 -->
   <link
     name="wheel_right_front_link">
@@ -220,5 +230,5 @@
           filename="package://jetrover_description/meshes/acker/wheel_right_front_link.stl" />
       </geometry>
-      <material name="black"/>
+      <material name="black" />
     </visual>
     <collision>
@@ -232,4 +242,5 @@
     </collision>
   </link>
+  <!-- 后前轮和底部钢板连接点 -->
   <joint
     name="wheel_right_front_joint"
@@ -245,4 +256,5 @@
       xyz="0 0 0" />
   </joint>
+  <!-- 右后轮 -->
   <link
     name="wheel_right_back_link">
@@ -269,5 +281,5 @@
           filename="package://jetrover_description/meshes/acker/wheel_right_back_link.stl" />
       </geometry>
-      <material name="black"/>
+      <material name="black" />
     </visual>
     <collision>
@@ -281,4 +293,5 @@
     </collision>
   </link>
+  <!-- 右后轮和底部钢板 联结 -->
   <joint
     name="wheel_right_back_joint"

File: src/jetrover_description/urdf/common.urdf.xacro (robot description, xacro)
@@ -1,4 +1,5 @@
 <?xml version="1.0" encoding="utf-8"?>
-<robot name="common" xmlns:xacro="http://ros.org/wiki/xacro" >
+<robot name="common" xmlns:xacro="http://ros.org/wiki/xacro">
+  <!-- 黑色保护罩 -->
   <link
     name="back_shell_black_link">
@@ -25,5 +26,5 @@
           filename="package://jetrover_description/meshes/common/back_shell_black_link.stl" />
       </geometry>
-      <material name="black"/>
+      <material name="black" />
     </visual>
     <collision>
@@ -37,4 +38,5 @@
     </collision>
   </link>
+  <!-- 黑色保护罩和车底钢板 联结 -->
   <joint
     name="back_shell_black_joint"
@@ -50,4 +52,5 @@
       xyz="0 0 0" />
   </joint>
+  <!-- 车顶钢板 -->
   <link
     name="back_shell_green_link">
@@ -74,5 +77,5 @@
           filename="package://jetrover_description/meshes/common/back_shell_green_link.stl" />
       </geometry>
-      <material name="green"/>
+      <material name="green" />
     </visual>
     <collision>
@@ -86,4 +89,5 @@
     </collision>
   </link>
+  <!-- 车顶钢板和车底钢板 联结 -->
   <joint
     name="back_shell_green_joint"

File: src/jetrover_description/urdf/connect.urdf.xacro (robot description, xacro)
@@ -2,4 +2,5 @@
 <robot name="arm" xmlns:xacro="http://ros.org/wiki/xacro">
   <xacro:property name="M_PI"   value="3.1415926535897931"/>
+  <!-- 第一节机械臂本体和车底钢板 联结 -->
   <joint
     name="joint1"

File: src/jetrover_description/urdf/depth_camera.urdf.xacro (robot description, xacro)
@@ -1,5 +1,6 @@
 <?xml version="1.0" encoding="utf-8"?>
-<robot name="depth_camera" xmlns:xacro="http://ros.org/wiki/xacro" >
-  <xacro:property name="M_PI"   value="3.1415926535897931"/>
+<robot name="depth_camera" xmlns:xacro="http://ros.org/wiki/xacro">
+  <xacro:property name="M_PI" value="3.1415926535897931" />
+  <!-- 相机底座 -->
   <link
     name="camera_connect_link">
@@ -26,5 +27,5 @@
           filename="package://jetrover_description/meshes/arm/camera_connect_link.STL" />
       </geometry>
-      <material name="black"/>
+      <material name="black" />
     </visual>
     <collision>
@@ -38,4 +39,5 @@
     </collision>
   </link>
+  <!-- 相机底座和机械臂4（从下往上数） 联结-->
   <joint
     name="camera_connect_joint"
@@ -51,4 +53,5 @@
       xyz="0 0 0" />
   </joint>
+  <!-- 相机本体 -->
   <link
     name="depth_cam_link">
@@ -91,4 +94,5 @@
     </collision>
   </link>
+  <!-- 相机本体和相机底座 联结-->
   <joint
     name="depth_cam_joint"
@@ -96,5 +100,5 @@
     <origin
       xyz="0 0.0 0.014475"
-      rpy="${M_PI} -${M_PI/2} -${M_PI/2}"/>
+      rpy="${M_PI} -${M_PI/2} -${M_PI/2}" />
     <parent
       link="camera_connect_link" />
@@ -104,5 +108,7 @@
       xyz="0 0 0" />
   </joint>
+  <!-- 相机坐标系 -->
   <link name="depth_cam_frame" />
+  <!-- 相机坐标系和相机本体 联结 -->
   <joint
     name="depth_cam_joint_sim"

File: src/jetrover_description/urdf/gripper.urdf.xacro (robot description, xacro)
@@ -1,5 +1,6 @@
 <?xml version="1.0" encoding="utf-8"?>
 <robot name="gripper" xmlns:xacro="http://ros.org/wiki/xacro">
-  <xacro:property name="M_PI"   value="3.1415926535897931"/>
+  <xacro:property name="M_PI" value="3.1415926535897931" />
+  <!-- 左夹爪 -->
   <link
     name="r_link">
@@ -26,5 +27,5 @@
           filename="package://jetrover_description/meshes/gripper/r_link.STL" />
       </geometry>
-      <material name="black"/>
+      <material name="black" />
     </visual>
     <collision>
@@ -38,4 +39,5 @@
     </collision>
   </link>
+  <!-- 左夹爪和夹爪底座 联结-->
   <joint
     name="r_joint"
@@ -56,4 +58,5 @@
       velocity="10" />
   </joint>
+  <!-- 右夹爪 -->
   <link
     name="l_link">
@@ -80,5 +83,5 @@
           filename="package://jetrover_description/meshes/gripper/l_link.STL" />
       </geometry>
-      <material name="black"/>
+      <material name="black" />
     </visual>
     <collision>
@@ -92,4 +95,5 @@
     </collision>
   </link>
+  <!-- 右夹爪和夹爪底座 联结 -->
   <joint
     name="l_joint"
@@ -114,4 +118,5 @@
       offset="0" />
   </joint>
+  <!-- 左夹爪支撑连杆 -->
   <link
     name="l_in_link">
@@ -138,5 +143,5 @@
           filename="package://jetrover_description/meshes/gripper/l_in_link.STL" />
       </geometry>
-      <material name="black"/>
+      <material name="black" />
     </visual>
     <collision>
@@ -150,4 +155,5 @@
     </collision>
   </link>
+  <!-- 左夹爪支撑力连杆和夹爪底座 联结 -->
   <joint
     name="l_in_joint"
@@ -172,4 +178,5 @@
       offset="0" />
   </joint>
+  <!-- 左手指 -->
   <link
     name="l_out_link">
@@ -196,5 +203,5 @@
           filename="package://jetrover_description/meshes/gripper/l_out_link.STL" />
       </geometry>
-      <material name="black"/>
+      <material name="black" />
     </visual>
     <collision>
@@ -208,4 +215,5 @@
     </collision>
   </link>
+  <!-- 左手指和左支撑连杆 联结 -->
   <joint
     name="l_out_joint"
@@ -230,4 +238,5 @@
       offset="0" />
   </joint>
+  <!-- 右支撑连杆 -->
   <link
     name="r_in_link">
@@ -254,5 +263,5 @@
           filename="package://jetrover_description/meshes/gripper/r_in_link.STL" />
       </geometry>
-      <material name="black"/>
+      <material name="black" />
     </visual>
     <collision>
@@ -266,4 +275,5 @@
     </collision>
   </link>
+  <!-- 右支撑连杆和夹爪底座 联结 -->
   <joint
     name="r_in_joint"
@@ -288,4 +298,5 @@
       offset="0" />
   </joint>
+  <!-- 右手指 -->
   <link
     name="r_out_link">
@@ -312,5 +323,5 @@
           filename="package://jetrover_description/meshes/gripper/r_out_link.STL" />
       </geometry>
-      <material name="black"/>
+      <material name="black" />
     </visual>
     <collision>
@@ -324,4 +335,5 @@
     </collision>
   </link>
+  <!-- 右手指和右支撑连杆 联结 -->
   <joint
     name="r_out_joint"

File: src/jetrover_description/urdf/imu.urdf.xacro (robot description, xacro)
@@ -2,4 +2,5 @@
 <robot name="imu" xmlns:xacro="http://ros.org/wiki/xacro">
   <xacro:property name="M_PI" value="3.1415926535897931"/>
+  <!-- IMU 本体 -->
   <link
     name="imu_link">
@@ -38,4 +39,5 @@
     </collision>
   </link>
+  <!-- IMU 本体和彻底钢板 联结 -->
   <joint
     name="imu_joint"

File: src/jetrover_description/urdf/jetrover.xacro (robot description, xacro)
@@ -1,14 +1,23 @@
 <?xml version="1.0" encoding="utf-8"?>
 <robot name="jetrover" xmlns:xacro="http://ros.org/wiki/xacro">
-    <xacro:include filename="$(find jetrover_description)/urdf/materials.xacro"/>
+    <xacro:include filename="$(find jetrover_description)/urdf/materials.xacro" />
     <xacro:include filename="$(find jetrover_description)/urdf/inertial_matrix.xacro" />
-    <xacro:include filename="$(find jetrover_description)/urdf/lidar_a1.urdf.xacro"/>
-    <xacro:include filename="$(find jetrover_description)/urdf/car_acker.urdf.xacro"/>
-    <xacro:include filename="$(find jetrover_description)/urdf/lidar.urdf.xacro"/>
-    <xacro:include filename="$(find jetrover_description)/urdf/imu.urdf.xacro"/>
-    <xacro:include filename="$(find jetrover_description)/urdf/depth_camera.urdf.xacro"/>
-    <xacro:include filename="$(find jetrover_description)/urdf/common.urdf.xacro"/>
-    <xacro:include filename="$(find jetrover_description)/urdf/connect.urdf.xacro"/>
-    <xacro:include filename="$(find jetrover_description)/urdf/arm.urdf.xacro"/>
-    <xacro:include filename="$(find jetrover_description)/urdf/gripper.urdf.xacro"/>
+    <!-- 车底&中间层钢板，车轮 -->
+    <xacro:include filename="$(find jetrover_description)/urdf/car_acker.urdf.xacro" />
+    <!-- 车顶钢板、车顶黑色保护罩 -->
+    <xacro:include filename="$(find jetrover_description)/urdf/common.urdf.xacro" />
+    <!-- A1 LiDAR 雷达和车底钢板 -->
+    <xacro:include filename="$(find jetrover_description)/urdf/lidar.urdf.xacro" />
+    <!-- A1 LiDAR 坐标系 和 A1 LiDAR 本体 -->
+    <xacro:include filename="$(find jetrover_description)/urdf/lidar_a1.urdf.xacro" />
+    <!-- IMU 本体和车底钢板 -->
+    <xacro:include filename="$(find jetrover_description)/urdf/imu.urdf.xacro" />
+    <!-- 相机坐标系，本体，底座 -->
+    <xacro:include filename="$(find jetrover_description)/urdf/depth_camera.urdf.xacro" />
+    <!-- 第一节机械臂和车底钢板 联结 -->
+    <xacro:include filename="$(find jetrover_description)/urdf/connect.urdf.xacro" />
+    <!-- 机械臂和机械臂末端坐标系 -->
+    <xacro:include filename="$(find jetrover_description)/urdf/arm.urdf.xacro" />
+    <!-- 夹爪构造 -->
+    <xacro:include filename="$(find jetrover_description)/urdf/gripper.urdf.xacro" />
 </robot>

File: src/jetrover_description/urdf/lidar.urdf.xacro (robot description, xacro)
@@ -2,4 +2,5 @@
 <robot name="lidar" xmlns:xacro="http://ros.org/wiki/xacro" >
   <xacro:property name="M_PI" value="3.1415926535897931"/>
+  <!-- A1 LiDAR 雷达本体 -->
   <link
     name="lidar_link">
@@ -38,4 +39,5 @@
     <!--</collision>-->
   </link>
+  <!-- A1 LiDAR 雷达本体和车底钢板 联结 -->
   <joint
     name="lidar_joint"

File: src/jetrover_description/urdf/lidar_a1.urdf.xacro (robot description, xacro)
@@ -2,5 +2,7 @@
 <robot name="lidar_a1" xmlns:xacro="http://ros.org/wiki/xacro" >
   <xacro:property name="M_PI" value="3.1415926535897931"/>
+  <!-- A1 LiDAR 坐标系 -->
   <link name="lidar_frame" />
+  <!-- A1 LiDAR 坐标系和 A1 LiDAR 雷达本体 联结 -->
   <joint
     name="lidar_frame_joint"
