Commit message: 添加rebuild机器人底盘description文件

File: src/jetrover_description/urdf/arm.urdf.xacro (robot description, xacro)
@@ -2,5 +2,4 @@
 <robot name="arm" xmlns:xacro="http://ros.org/wiki/xacro">
   <xacro:property name="M_PI"   value="3.1415926535897931"/>
-  <!-- 第一节机械臂本体 -->
   <link
     name="link1">
@@ -39,5 +38,4 @@
     </collision>
   </link>
-  <!-- 伺服电机1 -->
   <link
     name="servo_link1">
@@ -76,5 +74,4 @@
     </collision>
   </link>
-  <!-- 第一节机械臂和伺服电机1 联结 -->
   <joint
     name="servo_joint1"
@@ -90,5 +87,4 @@
       xyz="0 0 0" />
   </joint>
-  <!-- 第二节机械臂本体 -->
   <link
     name="link2">
@@ -127,5 +123,4 @@
     </collision>
   </link>
-  <!-- 第二节机械臂和伺服电机1 联结 -->
   <joint
     name="joint2"
@@ -146,5 +141,4 @@
       velocity="10" />
   </joint>
-  <!-- 第三节机械臂本体 -->
   <link
     name="link3">
@@ -183,5 +177,4 @@
     </collision>
   </link>
-  <!-- 第三节机械臂本体和第二节机械臂本体 联结 -->
   <joint
     name="joint3"
@@ -202,5 +195,4 @@
       velocity="10" />
   </joint>
-  <!-- 第四节机械臂本体 -->
   <link
     name="link4">
@@ -239,5 +231,4 @@
     </collision>
   </link>
-  <!-- 第三节机械臂和第四节机械臂 联结 -->
   <joint
     name="joint4"
@@ -258,5 +249,4 @@
       velocity="10" />
   </joint>
-  <!-- 伺服电机2 -->
   <link
     name="servo_link2">
@@ -295,5 +285,4 @@
     </collision>
   </link>
-  <!-- 第四节机械臂和伺服电机2 联结 -->
   <joint
     name="servo_joint2"
@@ -309,5 +298,4 @@
       xyz="0 0 0" />
   </joint>
-  <!-- 夹爪旋转垫片 -->
   <link
     name="link5">
@@ -346,5 +334,4 @@
     </collision>
   </link>
-  <!-- 夹爪旋转垫片和伺服电机2 联结 -->
   <joint
     name="joint5"
@@ -365,5 +352,4 @@
       velocity="10" />
   </joint>
-  <!-- 夹爪底座 -->
   <link
     name="gripper_link">
@@ -402,5 +388,4 @@
     </collision>
   </link>
-  <!-- 夹爪底座和夹爪旋转垫片 联结 -->
   <joint
     name="gripper_joint"
@@ -416,7 +401,6 @@
       xyz="0 0 0" />
   </joint>
-  <!-- 末端执行器（坐标系） -->
+  <!-- end effector link -->
   <link name="end_effector_link" />
-  <!-- 末端执行器（坐标系）和夹爪旋转垫片 联结 -->
   <joint name="end_effector_joint" type="fixed">
     <origin xyz="0 0 0.08" rpy="0 0 0"/>

File: src/jetrover_description/urdf/car_acker.urdf.xacro (robot description, xacro)
@@ -2,19 +2,42 @@
 <robot name="jetrover" xmlns:xacro="http://ros.org/wiki/xacro">
   <xacro:property name="M_PI" value="3.1415926535897931" />
-  <link name="base_footprint" />
   <xacro:property name="base_link_mass" value="1.6" />
   <xacro:property name="base_link_w" value="0.30" />
   <xacro:property name="base_link_h" value="0.15" />
   <xacro:property name="base_link_d" value="0.10" />
-  <!-- 车底钢板和垂直投影 联结 -->
+  <!-- 车底垂直投影地面中间处 -->
+  <link name="base_footprint" />
+  <!-- 底盘中间件上表面中心处 -->
+  <link name="base_link">
+    <xacro:box_inertial m="${base_link_mass}" w="${base_link_w}" h="${base_link_h}"
+      d="${base_link_d}" x="0" y="0" z="-0.15" />
+    <visual>
+      <origin
+        xyz="0 0 0"
+        rpy="0 0 0" />
+      <geometry>
+        <mesh
+          filename="package://jetrover_description/meshes/acker/base_link.stl" />
+      </geometry>
+      <material name="black" />
+    </visual>
+    <collision>
+      <origin
+        xyz="0 0 0"
+        rpy="0 0 0" />
+      <geometry>
+        <mesh
+          filename="package://jetrover_description/meshes/acker/base_link.stl" />
+      </geometry>
+    </collision>
+  </link>
   <joint name="base_joint" type="fixed">
-    <parent link="base_footprint" />   <!-- 机器人垂直投影到地面的坐标系 -->
+    <parent link="base_footprint" />
     <child link="base_link" />
     <origin xyz="0.0 0.0 ${0.05 + 0.0654867643253843}" rpy="0 0 0" />
   </joint>
+  <!-- 底盘中间件上表面中心处 -->
   <link name="w_link" />
-  <joint
-    name="w_joint"
-    type="fixed">
+  <joint name="w_joint" type="fixed">
     <origin
       xyz="0 0 0"
@@ -27,32 +50,6 @@
       xyz="0 0 0" />
   </joint>
-  <!-- 车底钢板 -->
-  <link
-    name="base_link">
-    <xacro:box_inertial m="${base_link_mass}" w="${base_link_w}" h="${base_link_h}"
-      d="${base_link_d}" x="0" y="0" z="-0.15" />
-    <visual>
-      <origin
-        xyz="0 0 0"
-        rpy="0 0 0" />
-      <geometry>
-        <mesh
-          filename="package://jetrover_description/meshes/acker/base_link.stl" />
-      </geometry>
-      <material name="black" />
-    </visual>
-    <collision>
-      <origin
-        xyz="0 0 0"
-        rpy="0 0 0" />
-      <geometry>
-        <mesh
-          filename="package://jetrover_description/meshes/acker/base_link.stl" />
-      </geometry>
-    </collision>
-  </link>
-  <!-- 车底中间层钢板 -->
-  <link
-    name="base_green_link">
+  <!-- 底盘中间件上表面中心处 -->
+  <link name="base_green_link">
     <inertial>
       <origin
@@ -89,8 +86,5 @@
     </collision>
   </link>
-  <!-- 车底钢板 中间夹层钢板 联结 -->
-  <joint
-    name="base_green_joint"
-    type="fixed">
+  <joint name="base_green_joint" type="fixed">
     <origin
       xyz="0 0 0"
@@ -104,12 +98,8 @@
   </joint>
   <!-- 左前轮 -->
-  <link
-    name="wheel_left_front_link">
-    <inertial>
-      <origin
-        xyz="-0.213334280297957 -0.203369638948946 -0.000334615151787748"
-        rpy="0 0 0" />
-      <mass
-        value="0.124188560741815" />
+  <link name="wheel_left_front_link">
+    <inertial>
+      <origin xyz="-0.213334280297957 -0.203369638948946 -0.000334615151787748" rpy="0 0 0" />
+      <mass value="0.124188560741815" />
       <inertia
         ixx="0.000108426797272382"
@@ -121,27 +111,18 @@
     </inertial>
     <visual>
-      <origin
-        xyz="0 0 0"
-        rpy="0 0 0" />
-      <geometry>
-        <mesh
-          filename="package://jetrover_description/meshes/acker/wheel_left_front_link.stl" />
-      </geometry>
-      <material name="black" />
-    </visual>
-    <collision>
-      <origin
-        xyz="0 0 0"
-        rpy="0 0 0" />
-      <geometry>
-        <mesh
-          filename="package://jetrover_description/meshes/acker/wheel_left_front_link.stl" />
-      </geometry>
-    </collision>
-  </link>
-  <!-- 左前轮和底部钢板 联结 -->
-  <joint
-    name="wheel_left_front_joint"
-    type="fixed">
+      <origin xyz="0 0 0" rpy="0 0 0" />
+      <geometry>
+        <mesh filename="package://jetrover_description/meshes/acker/wheel_left_front_link.stl" />
+      </geometry>
+      <material name="black" />
+    </visual>
+    <collision>
+      <origin xyz="0 0 0" rpy="0 0 0" />
+      <geometry>
+        <mesh filename="package://jetrover_description/meshes/acker/wheel_left_front_link.stl" />
+      </geometry>
+    </collision>
+  </link>
+  <joint name="wheel_left_front_joint" type="fixed">
     <origin
       xyz="-0.106579884267788 -0.0916974467397005 -0.0654867643253843"
@@ -154,7 +135,7 @@
       xyz="0 0 0" />
   </joint>
+  <!-- <link name="wheel_left_front_steering_link" /> -->
   <!-- 左后轮 -->
-  <link
-    name="wheel_left_back_link">
+  <link name="wheel_left_back_link">
     <inertial>
       <origin
@@ -191,8 +172,5 @@
     </collision>
   </link>
-  <!-- 左后轮和底部钢板 联结 -->
-  <joint
-    name="wheel_left_back_joint"
-    type="continuous">
+  <joint name="wheel_left_back_joint" type="fixed">
     <origin
       xyz="0.106753653016542 -0.0920004072996187 -0.0658214520621466"
@@ -203,9 +181,8 @@
       link="wheel_left_back_link" />
     <axis
-      xyz="0 1 0" />
+      xyz="0 0 0" />
   </joint>
   <!-- 右前轮 -->
-  <link
-    name="wheel_right_front_link">
+  <link name="wheel_right_front_link">
     <inertial>
       <origin
@@ -242,8 +219,5 @@
     </collision>
   </link>
-  <!-- 后前轮和底部钢板连接点 -->
-  <joint
-    name="wheel_right_front_joint"
-    type="fixed">
+  <joint name="wheel_right_front_joint" type="fixed">
     <origin
       xyz="-0.10658 0.091851 -0.065487"
@@ -256,7 +230,7 @@
       xyz="0 0 0" />
   </joint>
+  <!-- <link name="wheel_right_front_steering_link" /> -->
   <!-- 右后轮 -->
-  <link
-    name="wheel_right_back_link">
+  <link name="wheel_right_back_link">
     <inertial>
       <origin
@@ -293,8 +267,5 @@
     </collision>
   </link>
-  <!-- 右后轮和底部钢板 联结 -->
-  <joint
-    name="wheel_right_back_joint"
-    type="continuous">
+  <joint name="wheel_right_back_joint" type="fixed">
     <origin
       xyz="0.10675 0.091848 -0.065821"
@@ -305,6 +276,5 @@
       link="wheel_right_back_link" />
     <axis
-      xyz="0 1 0" />
-  </joint>
-  <!-- <xacro:include filename="$(find jetrover_description)/gazebo/car_acker_gazebo.xacro" /> -->
+      xyz="0 0 0" />
+  </joint>
 </robot>

File: src/jetrover_description/urdf/common.urdf.xacro (robot description, xacro)
@@ -1,5 +1,5 @@
 <?xml version="1.0" encoding="utf-8"?>
 <robot name="common" xmlns:xacro="http://ros.org/wiki/xacro">
-  <!-- 黑色保护罩 -->
+  <!-- 显示器保护壳连接体 -->
   <link
     name="back_shell_black_link">
@@ -38,5 +38,5 @@
     </collision>
   </link>
-  <!-- 黑色保护罩和车底钢板 联结 -->
+  <!-- 显示器保护壳连接体与底盘连接 -->
   <joint
     name="back_shell_black_joint"
@@ -52,5 +52,5 @@
       xyz="0 0 0" />
   </joint>
-  <!-- 车顶钢板 -->
+  <!-- 底盘结构上层组件 -->
   <link
     name="back_shell_green_link">
@@ -89,5 +89,5 @@
     </collision>
   </link>
-  <!-- 车顶钢板和车底钢板 联结 -->
+  <!-- 底盘结构上层组件与底盘连接 -->
   <joint
     name="back_shell_green_joint"

File: src/jetrover_description/urdf/connect.urdf.xacro (robot description, xacro)
@@ -2,5 +2,4 @@
 <robot name="arm" xmlns:xacro="http://ros.org/wiki/xacro">
   <xacro:property name="M_PI"   value="3.1415926535897931"/>
-  <!-- 第一节机械臂本体和车底钢板 联结 -->
   <joint
     name="joint1"

File: src/jetrover_description/urdf/depth_camera.urdf.xacro (robot description, xacro)
@@ -1,6 +1,5 @@
 <?xml version="1.0" encoding="utf-8"?>
-<robot name="depth_camera" xmlns:xacro="http://ros.org/wiki/xacro">
-  <xacro:property name="M_PI" value="3.1415926535897931" />
-  <!-- 相机底座 -->
+<robot name="depth_camera" xmlns:xacro="http://ros.org/wiki/xacro" >
+  <xacro:property name="M_PI"   value="3.1415926535897931"/>
   <link
     name="camera_connect_link">
@@ -27,5 +26,5 @@
           filename="package://jetrover_description/meshes/arm/camera_connect_link.STL" />
       </geometry>
-      <material name="black" />
+      <material name="black"/>
     </visual>
     <collision>
@@ -39,5 +38,4 @@
     </collision>
   </link>
-  <!-- 相机底座和机械臂4（从下往上数） 联结-->
   <joint
     name="camera_connect_joint"
@@ -53,5 +51,4 @@
       xyz="0 0 0" />
   </joint>
-  <!-- 相机本体 -->
   <link
     name="depth_cam_link">
@@ -94,5 +91,4 @@
     </collision>
   </link>
-  <!-- 相机本体和相机底座 联结-->
   <joint
     name="depth_cam_joint"
@@ -100,5 +96,5 @@
     <origin
       xyz="0 0.0 0.014475"
-      rpy="${M_PI} -${M_PI/2} -${M_PI/2}" />
+      rpy="${M_PI} -${M_PI/2} -${M_PI/2}"/>
     <parent
       link="camera_connect_link" />
@@ -108,7 +104,5 @@
       xyz="0 0 0" />
   </joint>
-  <!-- 相机坐标系 -->
   <link name="depth_cam_frame" />
-  <!-- 相机坐标系和相机本体 联结 -->
   <joint
     name="depth_cam_joint_sim"

File: src/jetrover_description/urdf/gripper.urdf.xacro (robot description, xacro)
@@ -1,6 +1,5 @@
 <?xml version="1.0" encoding="utf-8"?>
 <robot name="gripper" xmlns:xacro="http://ros.org/wiki/xacro">
-  <xacro:property name="M_PI" value="3.1415926535897931" />
-  <!-- 左夹爪 -->
+  <xacro:property name="M_PI"   value="3.1415926535897931"/>
   <link
     name="r_link">
@@ -27,5 +26,5 @@
           filename="package://jetrover_description/meshes/gripper/r_link.STL" />
       </geometry>
-      <material name="black" />
+      <material name="black"/>
     </visual>
     <collision>
@@ -39,5 +38,4 @@
     </collision>
   </link>
-  <!-- 左夹爪和夹爪底座 联结-->
   <joint
     name="r_joint"
@@ -58,5 +56,4 @@
       velocity="10" />
   </joint>
-  <!-- 右夹爪 -->
   <link
     name="l_link">
@@ -83,5 +80,5 @@
           filename="package://jetrover_description/meshes/gripper/l_link.STL" />
       </geometry>
-      <material name="black" />
+      <material name="black"/>
     </visual>
     <collision>
@@ -95,5 +92,4 @@
     </collision>
   </link>
-  <!-- 右夹爪和夹爪底座 联结 -->
   <joint
     name="l_joint"
@@ -118,5 +114,4 @@
       offset="0" />
   </joint>
-  <!-- 左夹爪支撑连杆 -->
   <link
     name="l_in_link">
@@ -143,5 +138,5 @@
           filename="package://jetrover_description/meshes/gripper/l_in_link.STL" />
       </geometry>
-      <material name="black" />
+      <material name="black"/>
     </visual>
     <collision>
@@ -155,5 +150,4 @@
     </collision>
   </link>
-  <!-- 左夹爪支撑力连杆和夹爪底座 联结 -->
   <joint
     name="l_in_joint"
@@ -178,5 +172,4 @@
       offset="0" />
   </joint>
-  <!-- 左手指 -->
   <link
     name="l_out_link">
@@ -203,5 +196,5 @@
           filename="package://jetrover_description/meshes/gripper/l_out_link.STL" />
       </geometry>
-      <material name="black" />
+      <material name="black"/>
     </visual>
     <collision>
@@ -215,5 +208,4 @@
     </collision>
   </link>
-  <!-- 左手指和左支撑连杆 联结 -->
   <joint
     name="l_out_joint"
@@ -238,5 +230,4 @@
       offset="0" />
   </joint>
-  <!-- 右支撑连杆 -->
   <link
     name="r_in_link">
@@ -263,5 +254,5 @@
           filename="package://jetrover_description/meshes/gripper/r_in_link.STL" />
       </geometry>
-      <material name="black" />
+      <material name="black"/>
     </visual>
     <collision>
@@ -275,5 +266,4 @@
     </collision>
   </link>
-  <!-- 右支撑连杆和夹爪底座 联结 -->
   <joint
     name="r_in_joint"
@@ -298,5 +288,4 @@
       offset="0" />
   </joint>
-  <!-- 右手指 -->
   <link
     name="r_out_link">
@@ -323,5 +312,5 @@
           filename="package://jetrover_description/meshes/gripper/r_out_link.STL" />
       </geometry>
-      <material name="black" />
+      <material name="black"/>
     </visual>
     <collision>
@@ -335,5 +324,4 @@
     </collision>
   </link>
-  <!-- 右手指和右支撑连杆 联结 -->
   <joint
     name="r_out_joint"

File: src/jetrover_description/urdf/imu.urdf.xacro (robot description, xacro)
@@ -2,5 +2,4 @@
 <robot name="imu" xmlns:xacro="http://ros.org/wiki/xacro">
   <xacro:property name="M_PI" value="3.1415926535897931"/>
-  <!-- IMU 本体 -->
   <link
     name="imu_link">
@@ -39,5 +38,4 @@
     </collision>
   </link>
-  <!-- IMU 本体和彻底钢板 联结 -->
   <joint
     name="imu_joint"

File: src/jetrover_description/urdf/inertial_matrix.xacro (robot description, xacro)
@@ -20,13 +20,13 @@
       <inertia
         ixx="${m*(3*r*r+h*h)/12}"
-        ixy = "0"
-        ixz = "0"
+        ixy="0"
+        ixz="0"
         iyy="${m*(3*r*r+h*h)/12}"
-        iyz = "0"
+        iyz="0"
         izz="${m*r*r/2}" />
     </inertial>
   </xacro:macro>
   <xacro:macro name="box_inertial" params="m w h d x y z">
-      <inertial>
+    <inertial>
       <origin
         xyz="${x} ${y} ${z}"
@@ -35,8 +35,8 @@
       <inertia
         ixx="${m*(h*h+d*d)/12}"
-        ixy = "0"
-        ixz = "0"
+        ixy="0"
+        ixz="0"
         iyy="${m*(w*w+d*d)/12}"
-        iyz = "0"
+        iyz="0"
         izz="${m*(w*w+h*h)/12}" />
     </inertial>

File: src/jetrover_description/urdf/jetrover.xacro (robot description, xacro)
@@ -3,21 +3,16 @@
     <xacro:include filename="$(find jetrover_description)/urdf/materials.xacro" />
     <xacro:include filename="$(find jetrover_description)/urdf/inertial_matrix.xacro" />
-    <!-- 车底&中间层钢板，车轮 -->
+    <!-- 激光雷达和底座 -->
+    <xacro:include filename="$(find jetrover_description)/urdf/lidar_a1.urdf.xacro" />
+    <xacro:include filename="$(find jetrover_description)/urdf/lidar.urdf.xacro" />
+    <!-- 车载传感器 -->
+    <xacro:include filename="$(find jetrover_description)/urdf/imu.urdf.xacro" />
+    <xacro:include filename="$(find jetrover_description)/urdf/depth_camera.urdf.xacro" />
+    <!-- 机械臂 -->
+    <xacro:include filename="$(find jetrover_description)/urdf/connect.urdf.xacro" />
+    <xacro:include filename="$(find jetrover_description)/urdf/arm.urdf.xacro" />
+    <xacro:include filename="$(find jetrover_description)/urdf/gripper.urdf.xacro" />
+    <!-- 底盘结构 -->
     <xacro:include filename="$(find jetrover_description)/urdf/car_acker.urdf.xacro" />
-    <!-- 车顶钢板、车顶黑色保护罩 -->
     <xacro:include filename="$(find jetrover_description)/urdf/common.urdf.xacro" />
-    <!-- A1 LiDAR 雷达和车底钢板 -->
-    <xacro:include filename="$(find jetrover_description)/urdf/lidar.urdf.xacro" />
-    <!-- A1 LiDAR 坐标系 和 A1 LiDAR 本体 -->
-    <xacro:include filename="$(find jetrover_description)/urdf/lidar_a1.urdf.xacro" />
-    <!-- IMU 本体和车底钢板 -->
-    <xacro:include filename="$(find jetrover_description)/urdf/imu.urdf.xacro" />
-    <!-- 相机坐标系，本体，底座 -->
-    <xacro:include filename="$(find jetrover_description)/urdf/depth_camera.urdf.xacro" />
-    <!-- 第一节机械臂和车底钢板 联结 -->
-    <xacro:include filename="$(find jetrover_description)/urdf/connect.urdf.xacro" />
-    <!-- 机械臂和机械臂末端坐标系 -->
-    <xacro:include filename="$(find jetrover_description)/urdf/arm.urdf.xacro" />
-    <!-- 夹爪构造 -->
-    <xacro:include filename="$(find jetrover_description)/urdf/gripper.urdf.xacro" />
 </robot>

File: src/jetrover_description/urdf/lidar.urdf.xacro (robot description, xacro)
@@ -2,5 +2,4 @@
 <robot name="lidar" xmlns:xacro="http://ros.org/wiki/xacro" >
   <xacro:property name="M_PI" value="3.1415926535897931"/>
-  <!-- A1 LiDAR 雷达本体 -->
   <link
     name="lidar_link">
@@ -29,15 +28,11 @@
       <material name="black"/>
     </visual>
-    <!--<collision>-->
-      <!--<origin-->
-        <!--xyz="0 0 0"-->
-        <!--rpy="0 0 0" />-->
-      <!--<geometry>-->
-        <!--<mesh-->
-          <!--filename="package://jetrover_description/meshes/common/lidar_link.stl" />-->
-      <!--</geometry>-->
-    <!--</collision>-->
+    <collision>
+      <origin xyz="0 0 0" rpy="0 0 0" />
+      <geometry>
+        <mesh filename="package://jetrover_description/meshes/common/lidar_link.stl" />
+      </geometry>
+    </collision>
   </link>
-  <!-- A1 LiDAR 雷达本体和车底钢板 联结 -->
   <joint
     name="lidar_joint"

File: src/jetrover_description/urdf/lidar_a1.urdf.xacro (robot description, xacro)
@@ -2,7 +2,5 @@
 <robot name="lidar_a1" xmlns:xacro="http://ros.org/wiki/xacro" >
   <xacro:property name="M_PI" value="3.1415926535897931"/>
-  <!-- A1 LiDAR 坐标系 -->
   <link name="lidar_frame" />
-  <!-- A1 LiDAR 坐标系和 A1 LiDAR 雷达本体 联结 -->
   <joint
     name="lidar_frame_joint"
