Commit message: Rework simulation control stack with updated ros2_control xacro, Gazebo launch, and controller YAML

File: src/jetrover_description/urdf/assembly_simulation.xacro (robot description, xacro)
@@ -18,5 +18,5 @@
           scale="0.001 0.001 0.001" />
       </geometry>
-      <material name="silver"/>
+      <material name="silver" />
     </visual>
     <collision name="base_link_collision">
@@ -43,5 +43,5 @@
           scale="0.001 0.001 0.001" />
       </geometry>
-      <material name="silver"/>
+      <material name="silver" />
     </visual>
     <collision name="front_left_sterring_link_collision">
@@ -69,5 +69,5 @@
           scale="0.001 0.001 0.001" />
       </geometry>
-      <material name="silver"/>
+      <material name="silver" />
     </visual>
     <collision name="rear_right_wheel_link_collision">
@@ -95,5 +95,5 @@
           scale="0.001 0.001 0.001" />
       </geometry>
-      <material name="silver"/>
+      <material name="silver" />
     </visual>
     <collision name="rear_right_wheel_tire_collision">
@@ -121,5 +121,5 @@
           scale="0.001 0.001 0.001" />
       </geometry>
-      <material name="silver"/>
+      <material name="silver" />
     </visual>
     <collision name="back_shell_green_link_collision">
@@ -146,5 +146,5 @@
           scale="0.001 0.001 0.001" />
       </geometry>
-      <material name="silver"/>
+      <material name="silver" />
     </visual>
     <collision name="back_shell_black_link_collision">
@@ -172,5 +172,5 @@
           scale="0.001 0.001 0.001" />
       </geometry>
-      <material name="silver"/>
+      <material name="silver" />
     </visual>
     <collision name="front_right_steering_link_collision">
@@ -198,5 +198,5 @@
           scale="0.001 0.001 0.001" />
       </geometry>
-      <material name="silver"/>
+      <material name="silver" />
     </visual>
     <collision name="rear_left_wheel_tire_collision">
@@ -224,5 +224,5 @@
           scale="0.001 0.001 0.001" />
       </geometry>
-      <material name="silver"/>
+      <material name="silver" />
     </visual>
     <collision name="rear_left_wheel_link_collision">
@@ -250,5 +250,5 @@
           scale="0.001 0.001 0.001" />
       </geometry>
-      <material name="silver"/>
+      <material name="silver" />
     </visual>
     <collision name="front_right_wheel_link_collision">
@@ -276,5 +276,5 @@
           scale="0.001 0.001 0.001" />
       </geometry>
-      <material name="silver"/>
+      <material name="silver" />
     </visual>
     <collision name="front_right_wheel_tire_collision">
@@ -302,5 +302,5 @@
           scale="0.001 0.001 0.001" />
       </geometry>
-      <material name="silver"/>
+      <material name="silver" />
     </visual>
     <collision name="front_left_wheel_link_collision">
@@ -328,5 +328,5 @@
           scale="0.001 0.001 0.001" />
       </geometry>
-      <material name="silver"/>
+      <material name="silver" />
     </visual>
     <collision name="front_left_wheel_tire_collision">
@@ -352,5 +352,5 @@
           scale="0.001 0.001 0.001" />
       </geometry>
-      <material name="silver"/>
+      <material name="silver" />
     </visual>
     <collision name="base_green_link_collision">
@@ -378,5 +378,5 @@
           scale="0.001 0.001 0.001" />
       </geometry>
-      <material name="silver"/>
+      <material name="silver" />
     </visual>
     <collision name="link3_collision">
@@ -404,5 +404,5 @@
           scale="0.001 0.001 0.001" />
       </geometry>
-      <material name="silver"/>
+      <material name="silver" />
     </visual>
     <collision name="link4_collision">
@@ -430,5 +430,5 @@
           scale="0.001 0.001 0.001" />
       </geometry>
-      <material name="silver"/>
+      <material name="silver" />
     </visual>
     <collision name="camera_connect_link_collision">
@@ -456,5 +456,5 @@
           scale="0.001 0.001 0.001" />
       </geometry>
-      <material name="silver"/>
+      <material name="silver" />
     </visual>
     <collision name="depth_cam_link_collision">
@@ -482,5 +482,5 @@
           scale="0.001 0.001 0.001" />
       </geometry>
-      <material name="silver"/>
+      <material name="silver" />
     </visual>
     <collision name="gripper_link_collision">
@@ -508,5 +508,5 @@
           scale="0.001 0.001 0.001" />
       </geometry>
-      <material name="silver"/>
+      <material name="silver" />
     </visual>
     <collision name="l_link_collision">
@@ -534,5 +534,5 @@
           scale="0.001 0.001 0.001" />
       </geometry>
-      <material name="silver"/>
+      <material name="silver" />
     </visual>
     <collision name="r_link_collision">
@@ -560,5 +560,5 @@
           scale="0.001 0.001 0.001" />
       </geometry>
-      <material name="silver"/>
+      <material name="silver" />
     </visual>
     <collision name="imu_link_collision">
@@ -586,5 +586,5 @@
           scale="0.001 0.001 0.001" />
       </geometry>
-      <material name="silver"/>
+      <material name="silver" />
     </visual>
     <collision name="lidar_link_collision">
@@ -612,5 +612,5 @@
           scale="0.001 0.001 0.001" />
       </geometry>
-      <material name="silver"/>
+      <material name="silver" />
     </visual>
     <collision name="link1_collision">
@@ -638,5 +638,5 @@
           scale="0.001 0.001 0.001" />
       </geometry>
-      <material name="silver"/>
+      <material name="silver" />
     </visual>
     <collision name="link2_collision">
@@ -664,5 +664,5 @@
           scale="0.001 0.001 0.001" />
       </geometry>
-      <material name="silver"/>
+      <material name="silver" />
     </visual>
     <collision name="link5_collision">
@@ -690,5 +690,5 @@
           scale="0.001 0.001 0.001" />
       </geometry>
-      <material name="silver"/>
+      <material name="silver" />
     </visual>
     <collision name="l_out_link_collision">
@@ -716,5 +716,5 @@
           scale="0.001 0.001 0.001" />
       </geometry>
-      <material name="silver"/>
+      <material name="silver" />
     </visual>
     <collision name="r_out_link_collision">
@@ -803,5 +803,5 @@
     <axis xyz="0.0 0.0 1.0" />
   </joint>
-    <joint name="front_left_wheel_joint" type="continuous">
+  <joint name="front_left_wheel_joint" type="continuous">
     <origin xyz="-6.069000000000102e-05 -0.0282411 -0.021359399999999997"
       rpy="1.5707943460843194 2.5718047893657596e-11 -3.1415796693364713" />

Commit message: feat(sim): add Gazebo sensing pipeline for depth camera and lidar perception
Build a complete simulation perception pipeline for future projects, so the
development order is explicit and easy to follow:

1. model the sensor frames in URDF
   - add virtual_depth_cam_frame as a fixed frame under depth_cam_link
   - keep sensor pose aligned with TF instead of applying sensor-only pose offsets

2. attach sensors in Gazebo
   - add rgbd_camera and gpu_lidar sensor setup
   - bind the depth camera to virtual_depth_cam_frame
   - keep sensor topics consistent for downstream bridge / RViz usage

3. bridge Gazebo topics to ROS 2
   - add ros_gz_bridge mappings for:
     /clock
     /camera/image
     /camera/depth_image
     /camera/camera_info
     /camera/points
     /scan
     /scan/points

4. improve RViz visualization for perception debugging
   - add TF / Image / PointCloud2 / LaserScan displays
   - expose camera image, depth point cloud, and lidar scan for verification

5. load custom Gazebo world
   - replace empty.sdf with gz_world.sdf in gazebo launch

Runtime order:
1. launch simulation environment:
   ros2 launch jetrover_description ros2_control_sim.launch.py

   Note:
   gazebo.launch.py can also start gz sim, but it does not configure RViz2,
   so visualization is less convenient.
   At startup the arm stays at the Zero pose and the depth camera points upward,
   so the arm must be moved to the perception pose first.

2. launch MoveIt and enable sim time:
   ros2 launch jetrover_moveit_config demo.launch.py
   ros2 param set /move_group use_sim_time true

   Note:
   without setting use_sim_time to true, the arm will not move correctly in Gazebo.

3. in the MotionPlanning RViz plugin:
   - set Goal State to DepthCamPerception
   - click Plan & Execute

4. once the depth camera reaches the horizontal perception pose,
   the corresponding PointCloud2 data of the target object can be observed
   in the other RViz instance.

File: src/jetrover_description/urdf/assembly_simulation.xacro (robot description, xacro)
@@ -467,4 +467,5 @@
     </collision>
   </link>
+  <link name="virtual_depth_cam_frame" />
   <link name="gripper_link">
     <inertial>
@@ -854,4 +855,9 @@
     <child link="depth_cam_link" />
   </joint>
+  <joint name="virtual_depth_cam_frame_joint" type="fixed">
+    <parent link="depth_cam_link" />
+    <child link="virtual_depth_cam_frame" />
+    <origin xyz="0 0.022 -0.03" rpy="0 1.57079632679 0" />
+  </joint>
   <joint name="joint5" type="revolute">
     <origin xyz="-0.00024036999984703656 -0.053884690000000006 -0.026603920000001377"

Commit message: 添加办公室场景

File: src/jetrover_description/urdf/assembly_simulation.xacro (robot description, xacro)
@@ -787,8 +787,8 @@
   <joint name="rear_right_wheel_joint" type="continuous">
     <origin xyz="-0.10209827 -0.09192406 0.00023524999999998463"
-      rpy="-1.5707963267948966 -0.0 -4.61955986574744e-33" />
+      rpy="1.5707963267948966 -0.0 -4.61955986574744e-33" />
     <parent link="base_link" />
     <child link="rear_right_wheel_link" />
-    <axis xyz="0.0 0.0 1.0" />
+    <axis xyz="0.0 0.0 -1.0" />
   </joint>
   <joint name="Rigid16" type="fixed">

Commit message: 修复设置nav2_goal后机器人无法移动

File: src/jetrover_description/urdf/assembly_simulation.xacro (robot description, xacro)
@@ -572,4 +572,5 @@
     </collision>
   </link>
+  <link name="lidar_frame" />
   <link name="lidar_link">
     <inertial>
@@ -900,4 +901,10 @@
     <child link="lidar_link" />
   </joint>
+  <joint name="lidar_frame_joint" type="fixed">
+    <origin xyz="0 -0.0244 -0.065"
+      rpy="0.0 0.0 0.0" />
+    <parent link="lidar_link" />
+    <child link="lidar_frame" />
+  </joint>
   <joint name="l_gripper_joint" type="fixed">
     <origin xyz="0.029998859999999964 -0.0002617999999999987 8.199999999991548e-07"
