Commit message: jetrover底盘Gz sim, ros2_control, RViz 仿真闭环

File: src/jetrover_description/urdf/acker/assembly_chasis.xacro (robot description, xacro)
@@ -1,309 +1,350 @@
-<?xml version="1.0" ?>
+<?xml version="1.0"?>
 <robot name="assembly_chasis" xmlns:xacro="http://www.ros.org/wiki/xacro">
-<xacro:include filename="$(find jetrover_description)/urdf/acker/materials.xacro" />
-<xacro:include filename="$(find jetrover_description)/urdf/acker/assembly_chasis.ros2control" />
-<xacro:include filename="$(find jetrover_description)/urdf/acker/assembly_chasis.gazebo" />
-<link name="base_link">
-  <inertial>
-    <origin xyz="-0.006798258215834958 0.0012157481048894814 0.03342103979861439" rpy="0 0 0"/>
-    <mass value="1.1948281829220548"/>
-    <inertia ixx="0.003173" iyy="0.010286" izz="0.013229" ixy="0.000139" iyz="-3.2e-05" ixz="0.000327"/>
-  </inertial>
-  <visual>
-    <origin xyz="0 0 0" rpy="0 0 0"/>
-    <geometry>
-      <mesh filename="file://$(find jetrover_description)/meshes/acker/base_link.stl" scale="0.001 0.001 0.001"/>
-    </geometry>
-    <material name="silver"/>
-  </visual>
-  <collision>
-    <origin xyz="0 0 0" rpy="0 0 0"/>
-    <geometry>
-      <mesh filename="file://$(find jetrover_description)/meshes/acker/base_link.stl" scale="0.001 0.001 0.001"/>
-    </geometry>
-  </collision>
-</link>
-<link name="base_green_link_1">
-  <inertial>
-    <origin xyz="-0.139137 -0.036613 -0.031235" rpy="0 0 0"/>
-    <mass value="0.0"/>
-    <inertia ixx="0.0" iyy="0.0" izz="0.0" ixy="0.0" iyz="0.0" ixz="0.0"/>
-  </inertial>
-  <visual>
-    <origin xyz="-0.139137 -0.036613 -0.031235" rpy="0 0 0"/>
-    <geometry>
-      <mesh filename="file://$(find jetrover_description)/meshes/acker/base_green_link_1.stl" scale="0.001 0.001 0.001"/>
-    </geometry>
-    <material name="silver"/>
-  </visual>
-  <collision>
-    <origin xyz="-0.139137 -0.036613 -0.031235" rpy="0 0 0"/>
-    <geometry>
-      <mesh filename="file://$(find jetrover_description)/meshes/acker/base_green_link_1.stl" scale="0.001 0.001 0.001"/>
-    </geometry>
-  </collision>
-</link>
-<link name="front_left_wheel_tire_1">
-  <inertial>
-    <origin xyz="5.640824710106962e-07 0.012800126968121384 -4.6788513696771616e-07" rpy="0 0 0"/>
-    <mass value="0.06316889720600809"/>
-    <inertia ixx="7.1e-05" iyy="0.000134" izz="7.1e-05" ixy="0.0" iyz="-0.0" ixz="-0.0"/>
-  </inertial>
-  <visual>
-    <origin xyz="-0.111171 -0.091924 -0.052595" rpy="0 0 0"/>
-    <geometry>
-      <mesh filename="file://$(find jetrover_description)/meshes/acker/front_left_wheel_tire_1.stl" scale="0.001 0.001 0.001"/>
-    </geometry>
-    <material name="silver"/>
-  </visual>
-  <collision>
-    <origin xyz="-0.111171 -0.091924 -0.052595" rpy="0 0 0"/>
-    <geometry>
-      <mesh filename="file://$(find jetrover_description)/meshes/acker/front_left_wheel_tire_1.stl" scale="0.001 0.001 0.001"/>
-    </geometry>
-  </collision>
-</link>
-<link name="front_left_wheel_link_1">
-  <inertial>
-    <origin xyz="5.640824710106962e-07 0.012800126968121384 -4.678851369468995e-07" rpy="0 0 0"/>
-    <mass value="1.0742550415244152"/>
-    <inertia ixx="0.000516" iyy="0.000914" izz="0.000516" ixy="0.0" iyz="-0.0" ixz="-0.0"/>
-  </inertial>
-  <visual>
-    <origin xyz="-0.111171 -0.091924 -0.052595" rpy="0 0 0"/>
-    <geometry>
-      <mesh filename="file://$(find jetrover_description)/meshes/acker/front_left_wheel_link_1.stl" scale="0.001 0.001 0.001"/>
-    </geometry>
-    <material name="silver"/>
-  </visual>
-  <collision>
-    <origin xyz="-0.111171 -0.091924 -0.052595" rpy="0 0 0"/>
-    <geometry>
-      <mesh filename="file://$(find jetrover_description)/meshes/acker/front_left_wheel_link_1.stl" scale="0.001 0.001 0.001"/>
-    </geometry>
-  </collision>
-</link>
-<link name="front_right_wheel_tire_1">
-  <inertial>
-    <origin xyz="4.752872217600457e-07 -0.012800057006835924 -3.494061506931212e-07" rpy="0 0 0"/>
-    <mass value="0.06316889720600809"/>
-    <inertia ixx="7.1e-05" iyy="0.000134" izz="7.1e-05" ixy="0.0" iyz="0.0" ixz="-0.0"/>
-  </inertial>
-  <visual>
-    <origin xyz="-0.111171 0.091924 -0.052595" rpy="0 0 0"/>
-    <geometry>
-      <mesh filename="file://$(find jetrover_description)/meshes/acker/front_right_wheel_tire_1.stl" scale="0.001 0.001 0.001"/>
-    </geometry>
-    <material name="silver"/>
-  </visual>
-  <collision>
-    <origin xyz="-0.111171 0.091924 -0.052595" rpy="0 0 0"/>
-    <geometry>
-      <mesh filename="file://$(find jetrover_description)/meshes/acker/front_right_wheel_tire_1.stl" scale="0.001 0.001 0.001"/>
-    </geometry>
-  </collision>
-</link>
-<link name="front_right_wheel_link_1">
-  <inertial>
-    <origin xyz="4.752872217600457e-07 -0.012800057006835924 -3.494061506723045e-07" rpy="0 0 0"/>
-    <mass value="1.0742550415244152"/>
-    <inertia ixx="0.000516" iyy="0.000914" izz="0.000516" ixy="0.0" iyz="-0.0" ixz="0.0"/>
-  </inertial>
-  <visual>
-    <origin xyz="-0.111171 0.091924 -0.052595" rpy="0 0 0"/>
-    <geometry>
-      <mesh filename="file://$(find jetrover_description)/meshes/acker/front_right_wheel_link_1.stl" scale="0.001 0.001 0.001"/>
-    </geometry>
-    <material name="silver"/>
-  </visual>
-  <collision>
-    <origin xyz="-0.111171 0.091924 -0.052595" rpy="0 0 0"/>
-    <geometry>
-      <mesh filename="file://$(find jetrover_description)/meshes/acker/front_right_wheel_link_1.stl" scale="0.001 0.001 0.001"/>
-    </geometry>
-  </collision>
-</link>
-<link name="rear_left_wheel_tire_1">
-  <inertial>
-    <origin xyz="-2.748838707072876e-07 0.012800399382812494 2.4570465088219473e-07" rpy="0 0 0"/>
-    <mass value="0.06316889720600809"/>
-    <inertia ixx="7.1e-05" iyy="0.000134" izz="7.1e-05" ixy="0.0" iyz="0.0" ixz="0.0"/>
-  </inertial>
-  <visual>
-    <origin xyz="0.102098 -0.091924 -0.054235" rpy="0 0 0"/>
-    <geometry>
-      <mesh filename="file://$(find jetrover_description)/meshes/acker/rear_left_wheel_tire_1.stl" scale="0.001 0.001 0.001"/>
-    </geometry>
-    <material name="silver"/>
-  </visual>
-  <collision>
-    <origin xyz="0.102098 -0.091924 -0.054235" rpy="0 0 0"/>
-    <geometry>
-      <mesh filename="file://$(find jetrover_description)/meshes/acker/rear_left_wheel_tire_1.stl" scale="0.001 0.001 0.001"/>
-    </geometry>
-  </collision>
-</link>
-<link name="rear_left_wheel_link_1">
-  <inertial>
-    <origin xyz="-2.748838707072876e-07 0.012800399382812494 2.457046509030114e-07" rpy="0 0 0"/>
-    <mass value="1.0742550415244152"/>
-    <inertia ixx="0.000516" iyy="0.000914" izz="0.000516" ixy="0.0" iyz="0.0" ixz="0.0"/>
-  </inertial>
-  <visual>
-    <origin xyz="0.102098 -0.091924 -0.054235" rpy="0 0 0"/>
-    <geometry>
-      <mesh filename="file://$(find jetrover_description)/meshes/acker/rear_left_wheel_link_1.stl" scale="0.001 0.001 0.001"/>
-    </geometry>
-    <material name="silver"/>
-  </visual>
-  <collision>
-    <origin xyz="0.102098 -0.091924 -0.054235" rpy="0 0 0"/>
-    <geometry>
-      <mesh filename="file://$(find jetrover_description)/meshes/acker/rear_left_wheel_link_1.stl" scale="0.001 0.001 0.001"/>
-    </geometry>
-  </collision>
-</link>
-<link name="rear_right_wheel_tire_1">
-  <inertial>
-    <origin xyz="-2.748838707072876e-07 -0.012800060845091277 2.4570465088219473e-07" rpy="0 0 0"/>
-    <mass value="0.06316889720600809"/>
-    <inertia ixx="7.1e-05" iyy="0.000134" izz="7.1e-05" ixy="0.0" iyz="0.0" ixz="0.0"/>
-  </inertial>
-  <visual>
-    <origin xyz="0.102098 0.091924 -0.054235" rpy="0 0 0"/>
-    <geometry>
-      <mesh filename="file://$(find jetrover_description)/meshes/acker/rear_right_wheel_tire_1.stl" scale="0.001 0.001 0.001"/>
-    </geometry>
-    <material name="silver"/>
-  </visual>
-  <collision>
-    <origin xyz="0.102098 0.091924 -0.054235" rpy="0 0 0"/>
-    <geometry>
-      <mesh filename="file://$(find jetrover_description)/meshes/acker/rear_right_wheel_tire_1.stl" scale="0.001 0.001 0.001"/>
-    </geometry>
-  </collision>
-</link>
-<link name="rear_right_wheel_link_1">
-  <inertial>
-    <origin xyz="-2.748838707072876e-07 -0.012800060845091277 2.457046509030114e-07" rpy="0 0 0"/>
-    <mass value="1.0742550415244152"/>
-    <inertia ixx="0.000516" iyy="0.000914" izz="0.000516" ixy="0.0" iyz="0.0" ixz="0.0"/>
-  </inertial>
-  <visual>
-    <origin xyz="0.102098 0.091924 -0.054235" rpy="0 0 0"/>
-    <geometry>
-      <mesh filename="file://$(find jetrover_description)/meshes/acker/rear_right_wheel_link_1.stl" scale="0.001 0.001 0.001"/>
-    </geometry>
-    <material name="silver"/>
-  </visual>
-  <collision>
-    <origin xyz="0.102098 0.091924 -0.054235" rpy="0 0 0"/>
-    <geometry>
-      <mesh filename="file://$(find jetrover_description)/meshes/acker/rear_right_wheel_link_1.stl" scale="0.001 0.001 0.001"/>
-    </geometry>
-  </collision>
-</link>
-<link name="front_left_sterring_link_1">
-  <inertial>
-    <origin xyz="-0.0040465918921842176 0.006035056500165253 0.019363639865389158" rpy="0 0 0"/>
-    <mass value="0.07976552705950153"/>
-    <inertia ixx="1.9e-05" iyy="2.2e-05" izz="2.6e-05" ixy="-4e-06" iyz="-1e-06" ixz="-3e-06"/>
-  </inertial>
-  <visual>
-    <origin xyz="-0.111232 -0.063683 -0.031235" rpy="0 0 0"/>
-    <geometry>
-      <mesh filename="file://$(find jetrover_description)/meshes/acker/front_left_sterring_link_1.stl" scale="0.001 0.001 0.001"/>
-    </geometry>
-    <material name="silver"/>
-  </visual>
-  <collision>
-    <origin xyz="-0.111232 -0.063683 -0.031235" rpy="0 0 0"/>
-    <geometry>
-      <mesh filename="file://$(find jetrover_description)/meshes/acker/front_left_sterring_link_1.stl" scale="0.001 0.001 0.001"/>
-    </geometry>
-  </collision>
-</link>
-<link name="front_right_steering_link_1">
-  <inertial>
-    <origin xyz="-0.004058391449346527 -0.006054828705959386 0.019322305399745048" rpy="0 0 0"/>
-    <mass value="0.07950209290283795"/>
-    <inertia ixx="1.9e-05" iyy="2.2e-05" izz="2.6e-05" ixy="4e-06" iyz="1e-06" ixz="-3e-06"/>
-  </inertial>
-  <visual>
-    <origin xyz="-0.111232 0.063683 -0.031235" rpy="0 0 0"/>
-    <geometry>
-      <mesh filename="file://$(find jetrover_description)/meshes/acker/front_right_steering_link_1.stl" scale="0.001 0.001 0.001"/>
-    </geometry>
-    <material name="silver"/>
-  </visual>
-  <collision>
-    <origin xyz="-0.111232 0.063683 -0.031235" rpy="0 0 0"/>
-    <geometry>
-      <mesh filename="file://$(find jetrover_description)/meshes/acker/front_right_steering_link_1.stl" scale="0.001 0.001 0.001"/>
-    </geometry>
-  </collision>
-</link>
-<joint name="Rigid 1" type="fixed">
-  <origin xyz="0.139137 0.036613 0.031235" rpy="0 0 0"/>
-  <parent link="base_link"/>
-  <child link="base_green_link_1"/>
-</joint>
-<joint name="front_left_wheel_tire_rigid" type="fixed">
-  <origin xyz="0.0 0.0 0.0" rpy="0 0 0"/>
-  <parent link="front_left_wheel_link_1"/>
-  <child link="front_left_wheel_tire_1"/>
-</joint>
-<joint name="front_left_wheel_joint" type="continuous">
-  <origin xyz="-6.1e-05 0.028241 0.02136" rpy="0 0 0"/>
-  <parent link="front_left_sterring_link_1"/>
-  <child link="front_left_wheel_link_1"/>
-  <axis xyz="-7e-06 -1.0 9e-06"/>
-</joint>
-<joint name="front_right_wheel_tire_rigid" type="fixed">
-  <origin xyz="0.0 0.0 0.0" rpy="0 0 0"/>
-  <parent link="front_right_wheel_link_1"/>
-  <child link="front_right_wheel_tire_1"/>
-</joint>
-<joint name="front_right_wheel_joint" type="continuous">
-  <origin xyz="-6.1e-05 -0.028241 0.02136" rpy="0 0 0"/>
-  <parent link="front_right_steering_link_1"/>
-  <child link="front_right_wheel_link_1"/>
-  <axis xyz="0.0 1.0 0.0"/>
-</joint>
-<joint name="rear_left_wheel_tire_rigid" type="fixed">
-  <origin xyz="0.0 0.0 0.0" rpy="0 0 0"/>
-  <parent link="rear_left_wheel_link_1"/>
-  <child link="rear_left_wheel_tire_1"/>
-</joint>
-<joint name="rear_left_wheel_joint" type="continuous">
-  <origin xyz="-0.102098 0.091924 0.054235" rpy="0 0 0"/>
-  <parent link="base_link"/>
-  <child link="rear_left_wheel_link_1"/>
-  <axis xyz="0.0 1.0 0.0"/>
-</joint>
-<joint name="rear_right_wheel_tire_rigid" type="fixed">
-  <origin xyz="0.0 0.0 0.0" rpy="0 0 0"/>
-  <parent link="rear_right_wheel_link_1"/>
-  <child link="rear_right_wheel_tire_1"/>
-</joint>
-<joint name="rear_right_wheel_joint" type="continuous">
-  <origin xyz="-0.102098 -0.091924 0.054235" rpy="0 0 0"/>
-  <parent link="base_link"/>
-  <child link="rear_right_wheel_link_1"/>
-  <axis xyz="-0.0 -1.0 0.0"/>
-</joint>
-<joint name="front_left_steering_joint" type="revolute">
-  <origin xyz="0.111232 0.063683 0.031235" rpy="0 0 0"/>
-  <parent link="base_link"/>
-  <child link="front_left_sterring_link_1"/>
-  <axis xyz="0.0 0.0 -1.0"/>
-  <limit upper="0.645772" lower="-0.401426" effort="100" velocity="100"/>
-</joint>
-<joint name="front_right_steering_joint" type="revolute">
-  <origin xyz="0.111232 -0.063683 0.031235" rpy="0 0 0"/>
-  <parent link="base_link"/>
-  <child link="front_right_steering_link_1"/>
-  <axis xyz="0.0 0.0 -1.0"/>
-  <limit upper="0.401426" lower="-0.645772" effort="100" velocity="100"/>
-</joint>
+  <xacro:include filename="$(find jetrover_description)/urdf/acker/materials.xacro" />
+  <xacro:include filename="$(find jetrover_description)/urdf/acker/assembly_chasis.ros2control" />
+  <xacro:include filename="$(find jetrover_description)/urdf/acker/assembly_chasis.gazebo" />
+  <link name="base_link">
+    <inertial>
+      <origin xyz="-0.006798258215834958 0.0012157481048894814 0.03342103979861439" rpy="0 0 0" />
+      <mass value="1.1948281829220548" />
+      <inertia ixx="0.003173" iyy="0.010286" izz="0.013229" ixy="0.000139" iyz="-3.2e-05"
+        ixz="0.000327" />
+    </inertial>
+    <visual>
+      <origin xyz="0 0 0" rpy="0 0 0" />
+      <geometry>
+        <mesh filename="file://$(find jetrover_description)/meshes/acker/base_link.stl"
+          scale="0.001 0.001 0.001" />
+      </geometry>
+      <material name="silver" />
+    </visual>
+    <collision>
+      <origin xyz="0 0 0" rpy="0 0 0" />
+      <geometry>
+        <mesh filename="file://$(find jetrover_description)/meshes/acker/base_link.stl"
+          scale="0.001 0.001 0.001" />
+      </geometry>
+    </collision>
+  </link>
+  <link name="base_green_link_1">
+    <inertial>
+      <origin xyz="-0.139137 -0.036613 -0.031235" rpy="0 0 0" />
+      <mass value="0.0" />
+      <inertia ixx="0.0" iyy="0.0" izz="0.0" ixy="0.0" iyz="0.0" ixz="0.0" />
+    </inertial>
+    <visual>
+      <origin xyz="-0.139137 -0.036613 -0.031235" rpy="0 0 0" />
+      <geometry>
+        <mesh filename="file://$(find jetrover_description)/meshes/acker/base_green_link_1.stl"
+          scale="0.001 0.001 0.001" />
+      </geometry>
+      <material name="silver" />
+    </visual>
+    <collision>
+      <origin xyz="-0.139137 -0.036613 -0.031235" rpy="0 0 0" />
+      <geometry>
+        <mesh filename="file://$(find jetrover_description)/meshes/acker/base_green_link_1.stl"
+          scale="0.001 0.001 0.001" />
+      </geometry>
+    </collision>
+  </link>
+  <link name="front_left_wheel_tire_1">
+    <inertial>
+      <origin xyz="5.640824710106962e-07 0.012800126968121384 -4.6788513696771616e-07" rpy="0 0 0" />
+      <mass value="0.06316889720600809" />
+      <inertia ixx="7.1e-05" iyy="0.000134" izz="7.1e-05" ixy="0.0" iyz="-0.0" ixz="-0.0" />
+    </inertial>
+    <visual>
+      <origin xyz="-0.111171 -0.091924 -0.052595" rpy="0 0 0" />
+      <geometry>
+        <mesh
+          filename="file://$(find jetrover_description)/meshes/acker/front_left_wheel_tire_1.stl"
+          scale="0.001 0.001 0.001" />
+      </geometry>
+      <material name="silver" />
+    </visual>
+    <collision>
+      <origin xyz="-0.111171 -0.091924 -0.052595" rpy="0 0 0" />
+      <geometry>
+        <mesh
+          filename="file://$(find jetrover_description)/meshes/acker/front_left_wheel_tire_1.stl"
+          scale="0.001 0.001 0.001" />
+      </geometry>
+    </collision>
+  </link>
+  <link name="front_left_wheel_link_1">
+    <inertial>
+      <origin xyz="5.640824710106962e-07 0.012800126968121384 -4.678851369468995e-07" rpy="0 0 0" />
+      <mass value="1.0742550415244152" />
+      <inertia ixx="0.000516" iyy="0.000914" izz="0.000516" ixy="0.0" iyz="-0.0" ixz="-0.0" />
+    </inertial>
+    <visual>
+      <origin xyz="-0.111171 -0.091924 -0.052595" rpy="0 0 0" />
+      <geometry>
+        <mesh
+          filename="file://$(find jetrover_description)/meshes/acker/front_left_wheel_link_1.stl"
+          scale="0.001 0.001 0.001" />
+      </geometry>
+      <material name="silver" />
+    </visual>
+    <collision>
+      <origin xyz="-0.111171 -0.091924 -0.052595" rpy="0 0 0" />
+      <geometry>
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